File: CAN.kicad_sch (KiCad schematic)
At the start: 14 parts, among them U2 TJA1051T-3, U3 TJA1051T-3

Commit message: All 0603 version
Parts:
- C5, C6, C7, C8: footprint Capacitor_SMD:C_0402_1005Metric -> Capacitor_SMD:C_0603_1608Metric
- D1, D2: footprint LED_SMD:LED_0402_1005Metric -> LED_SMD:LED_0603_1608Metric
- R4, R5, R6, R7: footprint Resistor_SMD:R_0402_1005Metric -> Resistor_SMD:R_0603_1608Metric
Changed lines of the file:
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@@
       (effects (font (size 1.27 1.27)) (justify right))
     )
-    (property "Footprint" "LED_SMD:LED_0402_1005Metric" (at 102.616 88.138 0)
+    (property "Footprint" "LED_SMD:LED_0603_1608Metric" (at 102.616 88.138 0)
       (effects (font (size 1.27 1.27)) hide)
     )
@@
       (effects (font (size 1.27 1.27)) (justify right))
     )
-    (property "Footprint" "Resistor_SMD:R_0402_1005Metric" (at 102.616 80.518 0)
+    (property "Footprint" "Resistor_SMD:R_0603_1608Metric" (at 102.616 80.518 0)
       (effects (font (size 1.27 1.27)) hide)
     )
@@
       (effects (font (size 1.27 1.27)) (justify left))
     )
-    (property "Footprint" "Capacitor_SMD:C_0402_1005Metric" (at 114.808 88.773 0)
+    (property "Footprint" "Capacitor_SMD:C_0603_1608Metric" (at 114.808 88.773 0)
       (effects (font (size 1.27 1.27)) hide)
     )
@@
       (effects (font (size 1.27 1.27)) (justify right))
     )
-    (property "Footprint" "Resistor_SMD:R_0402_1005Metric" (at 103.759 117.602 0)
+    (property "Footprint" "Resistor_SMD:R_0603_1608Metric" (at 103.759 117.602 0)
       (effects (font (size 1.27 1.27)) hide)
     )
@@
       (effects (font (size 1.27 1.27)) (justify left))
     )
-    (property "Footprint" "Capacitor_SMD:C_0402_1005Metric" (at 115.062 124.841 0)
+    (property "Footprint" "Capacitor_SMD:C_0603_1608Metric" (at 115.062 124.841 0)
       (effects (font (size 1.27 1.27)) hide)
     )
@@
       (effects (font (size 1.27 1.27)) (justify left))
     )
-    (property "Footprint" "Capacitor_SMD:C_0402_1005Metric" (at 124.714 124.841 0)
+    (property "Footprint" "Capacitor_SMD:C_0603_1608Metric" (at 124.714 124.841 0)
       (effects (font (size 1.27 1.27)) hide)
     )
@@
       (effects (font (size 1.27 1.27)) (justify left))
     )
-    (property "Footprint" "Resistor_SMD:R_0402_1005Metric" (at 169.672 81.661 0)
+    (property "Footprint" "Resistor_SMD:R_0603_1608Metric" (at 169.672 81.661 0)
       (effects (font (size 1.27 1.27)) hide)
     )
@@
       (effects (font (size 1.27 1.27)) (justify left))
     )
-    (property "Footprint" "Capacitor_SMD:C_0402_1005Metric" (at 124.46 88.773 0)
+    (property "Footprint" "Capacitor_SMD:C_0603_1608Metric" (at 124.46 88.773 0)
       (effects (font (size 1.27 1.27)) hide)
     )
@@
       (effects (font (size 1.27 1.27)) (justify right))
     )
-    (property "Footprint" "LED_SMD:LED_0402_1005Metric" (at 103.759 126.238 0)
+    (property "Footprint" "LED_SMD:LED_0603_1608Metric" (at 103.759 126.238 0)
       (effects (font (size 1.27 1.27)) hide)
     )
@@
       (effects (font (size 1.27 1.27)) (justify left))
     )
-    (property "Footprint" "Resistor_SMD:R_0402_1005Metric" (at 169.672 117.221 0)
-      (effects (font (size 1.27 1.27)) hide)
-    )
+    (property "Footprint" "Resistor_SMD:R_0603_1608Metric" (at 169.672 117.221 0)
+      (effects (font (size 1.27 1.27)) hide)
+    )
