File: POWER.kicad_sch (KiCad schematic)
At the start: 13 parts, among them J2 Conn_01x04, J3 Conn_01x04, J4 Conn_01x02, U1 SY8303AAIC

Commit message: All 0603 version
Parts:
- C2, C3: footprint Capacitor_SMD:C_0402_1005Metric -> Capacitor_SMD:C_0603_1608Metric
- R1, R2, R3: footprint Resistor_SMD:R_0402_1005Metric -> Resistor_SMD:R_0603_1608Metric
Changed lines of the file:
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@@
       (effects (font (size 1.27 1.27)))
     )
-    (property "Footprint" "Capacitor_SMD:C_0402_1005Metric" (at 123.19 50.5968 0)
+    (property "Footprint" "Capacitor_SMD:C_0603_1608Metric" (at 123.19 50.5968 0)
       (effects (font (size 1.27 1.27)) hide)
     )
@@
       (effects (font (size 1.27 1.27)) (justify left))
     )
-    (property "Footprint" "Resistor_SMD:R_0402_1005Metric" (at 137.922 63.627 90)
+    (property "Footprint" "Resistor_SMD:R_0603_1608Metric" (at 137.922 63.627 90)
       (effects (font (size 1.27 1.27)) hide)
     )
@@
       (effects (font (size 1.27 1.27)) (justify right))
     )
-    (property "Footprint" "Resistor_SMD:R_0402_1005Metric" (at 141.478 76.327 90)
+    (property "Footprint" "Resistor_SMD:R_0603_1608Metric" (at 141.478 76.327 90)
       (effects (font (size 1.27 1.27)) hide)
     )
@@
       (effects (font (size 1.27 1.27)) (justify right))
     )
-    (property "Footprint" "Capacitor_SMD:C_0402_1005Metric" (at 145.0848 59.817 0)
+    (property "Footprint" "Capacitor_SMD:C_0603_1608Metric" (at 145.0848 59.817 0)
       (effects (font (size 1.27 1.27)) hide)
     )
@@
       (effects (font (size 1.27 1.27)) (justify right))
     )
-    (property "Footprint" "Resistor_SMD:R_0402_1005Metric" (at 128.778 76.327 90)
-      (effects (font (size 1.27 1.27)) hide)
-    )
+    (property "Footprint" "Resistor_SMD:R_0603_1608Metric" (at 128.778 76.327 90)
+      (effects (font (size 1.27 1.27)) hide)
+    )
