File: EtherCAT_FUNC.kicad_sch (KiCad schematic)
At the start: 24 parts, among them J1 axt430124, J2 Conn_01x02, J3 Conn_01x02, J4 Conn_01x04, J8 Conn_01x03, J9 Conn_01x08, U6 ESDS314

Commit message: Change conns of GPIO
Parts:
- removed J9: Conn_01x08, Connector_PinHeader_2.54mm:PinHeader_1x08_P2.54mm_Vertical, symbol Connector_Generic:Conn_01x08
- added J10, J11, J12, J13, J14, J15, J16, J9: Conn_01x02, Connector_JST:JST_GH_BM02B-GHS-TBT_1x02-1MP_P1.25mm_Vertical, symbol Connector_Generic:Conn_01x02
- H4, H5, H6, H7: footprint MountingHole:MountingHole_2.7mm_M2.5 -> EXTRA IC:M1.6
Connections:
- net GND: now also J10.1 (Pin_1), J11.1 (Pin_1), J12.1 (Pin_1), J13.1 (Pin_1), J14.1 (Pin_1), J15.1 (Pin_1), J16.1 (Pin_1), J9.1 (Pin_1)
- net GPIO1: now also J9.2 (Pin_2)
- net GPIO2: now also J10.2 (Pin_2)
- net GPIO3: now also J11.2 (Pin_2)
- net GPIO4: now also J12.2 (Pin_2)
- net GPIO5: now also J13.2 (Pin_2)
- net GPIO6: now also J14.2 (Pin_2)
- net GPIO7: now also J15.2 (Pin_2)
- net GPIO8: now also J16.2 (Pin_2)

Commit message: Change footprints of M2 and axt330124
Parts:
- J1: footprint EXTRA IC:axt430124 -> EXTRA IC:axt330124
Changed lines of the file:
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@@
       (effects (font (size 1.27 1.27)))
     )
-    (property "Footprint" "EXTRA IC:axt430124" (at 170.688 98.806 0)
+    (property "Footprint" "EXTRA IC:axt330124" (at 170.688 98.806 0)
       (effects (font (size 1.27 1.27)) hide)
     )

Commit message: All 0603 version
Parts:
- D1: footprint LED_SMD:LED_0402_1005Metric -> LED_SMD:LED_0603_1608Metric
- R4: footprint Resistor_SMD:R_0402_1005Metric -> Resistor_SMD:R_0603_1608Metric
Connections:
- net GND: now also J10.2 (Pin_2), J11.2 (Pin_2), J12.2 (Pin_2), J13.2 (Pin_2), J14.2 (Pin_2), J15.2 (Pin_2), J16.2 (Pin_2), J9.2 (Pin_2); no longer J10.1 (Pin_1), J11.1 (Pin_1), J12.1 (Pin_1), J13.1 (Pin_1), J14.1 (Pin_1), J15.1 (Pin_1), J16.1 (Pin_1), J9.1 (Pin_1)
- net GPIO1: now also J9.1 (Pin_1); no longer J9.2 (Pin_2)
- net GPIO2: now also J10.1 (Pin_1); no longer J10.2 (Pin_2)
- net GPIO3: now also J11.1 (Pin_1); no longer J11.2 (Pin_2)
- net GPIO4: now also J12.1 (Pin_1); no longer J12.2 (Pin_2)
- net GPIO5: now also J13.1 (Pin_1); no longer J13.2 (Pin_2)
- net GPIO6: now also J14.1 (Pin_1); no longer J14.2 (Pin_2)
- net GPIO7: now also J15.1 (Pin_1); no longer J15.2 (Pin_2)
- net GPIO8: now also J16.1 (Pin_1); no longer J16.2 (Pin_2)

Commit message: Official version
Parts:
- added H10: MountingHole, EXTRA IC:M1.6, symbol Mechanical:MountingHole
- H4, H5, H6, H7: footprint EXTRA IC:M1.6 -> EXTRA IC:M2_HOLE
- H8, H9: footprint EXTRA IC:M2 -> EXTRA IC:M2_noHOLE
Connections:
- net 3V3: no longer J1.22
- net GND: now also J1.23, J10.1 (Pin_1), J11.1 (Pin_1), J12.1 (Pin_1), J13.1 (Pin_1), J14.1 (Pin_1), J15.1 (Pin_1), J16.1 (Pin_1), J9.1 (Pin_1); no longer J10.2 (Pin_2), J11.2 (Pin_2), J12.2 (Pin_2), J13.2 (Pin_2), J14.2 (Pin_2), J15.2 (Pin_2), J16.2 (Pin_2), J9.2 (Pin_2)
- net GPIO1: now also J9.2 (Pin_2); no longer J9.1 (Pin_1)
- net GPIO2: now also J10.2 (Pin_2); no longer J10.1 (Pin_1)
- net GPIO3: now also J11.2 (Pin_2); no longer J11.1 (Pin_1)
- net GPIO4: now also J12.2 (Pin_2); no longer J12.1 (Pin_1)
- net GPIO5: now also J13.2 (Pin_2); no longer J13.1 (Pin_1)
- net GPIO6: now also J14.2 (Pin_2); no longer J14.1 (Pin_1)
- net GPIO7: now also J15.2 (Pin_2); no longer J15.1 (Pin_1)
- net GPIO8: now also J16.2 (Pin_2); no longer J16.1 (Pin_1)
- net LED_CAN0: now also J1.22; no longer J1.23
Other:
- moved on the sheet: J4, J8, U6
